Commit message: first

File: cakin_ws/src/my_robot/urdf/my_robot.xacro (robot description, xacro)
@@ -135,4 +135,11 @@
     </visual>
   </link>
+<joint name="camera_optical_joint" type="fixed">
+    <origin xyz="0 0 0" rpy="-1.5707 0 -1.5707"/>
+    <parent link="camera"/>
+    <child link="camera_link_optical"/>
+  </joint>
+  <link name="camera_link_optical">
+  </link>
   <joint type="fixed" name="hokuyo_joint">
     <origin xyz="0.05 0 0.08" rpy="0 0 0"/>
